File: hw/faux-pi-0.kicad_sch (KiCad schematic)
At the start: 59 parts, among them J1 PWR_IN, J10 USB, J2 DEBUG, J3 RUN, J6 HDMI_C_1.4, J8 GPIO, J9 Micro_SD_Card_Det, SW1 RESET, SW2 BOOTSEL, U1 RP2040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

Commit message: tweaks
Parts:
- renumbered JP3 to JP2, JP7 to JP3, JP8 to JP4, JP9 to JP5
Connections:
- net MISO0 renamed SPI0_POCI0
- net MOSI0 renamed SPI0_PICO0
Other:
- note added: "DANGER: Closing JP4 and JP5 connects 5V pullups on pins 27 and 28 of the GPIO header. Only do this if you know what you're doing!"
- note removed: "DANGER: Closing DVI_SCL and DVI_SDA enabels 5V pullups on pins 27 and 28 of the GPIO header. Only do this if you know what you're doing!"
Changed lines of the file:
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@@
     (stroke (width 0) (type default) (color 0 0 0 0))
   )
-  (wire (pts (xy 36.83 160.02) (xy 50.8 160.02))
+  (wire (pts (xy 36.83 161.29) (xy 50.8 161.29))
     (stroke (width 0) (type default) (color 0 0 0 0))
   )
@@
     (stroke (width 0) (type default) (color 0 0 0 0))
   )
-  (wire (pts (xy 78.74 160.02) (xy 92.71 160.02))
+  (wire (pts (xy 78.74 161.29) (xy 92.71 161.29))
     (stroke (width 0) (type default) (color 0 0 0 0))
   )
@@
     (stroke (width 0) (type default) (color 0 0 0 0))
   )
+  (wire (pts (xy 92.71 161.29) (xy 92.71 160.02))
+    (stroke (width 0) (type default) (color 0 0 0 0))
+  )
   (wire (pts (xy 331.47 213.36) (xy 331.47 212.09))
     (stroke (width 0) (type default) (color 0 0 0 0))
@@
     (stroke (width 0) (type default) (color 0 0 0 0))
   )
+  (wire (pts (xy 50.8 161.29) (xy 50.8 160.02))
+    (stroke (width 0) (type default) (color 0 0 0 0))
+  )
   (wire (pts (xy 62.23 100.33) (xy 62.23 101.6))
     (stroke (width 0) (type default) (color 0 0 0 0))
@@
     (effects (font (size 1.27 1.27)) (justify left bottom))
   )
-  (text "DANGER: Closing DVI_SCL and DVI_SDA enabels 5V pullups\non pins 27 and 28 of the GPIO header.  Only do this if\nyou know what you're doing!"
-    (at 281.94 100.33 0)
+  (text "DANGER: Closing JP4 and JP5 connects 5V pullups on pins 27 and 28\nof the GPIO header.  Only do this if you know what you're doing!"
+    (at 279.4 105.41 0)
     (effects (font (size 2 2)) (justify left bottom))
   )
@@
     (effects (font (size 1.27 1.27)) (justify right bottom))
   )
-  (label "MOSI0" (at 110.49 77.47 180)
+  (label "SPI0_PICO0" (at 110.49 77.47 180)
     (effects (font (size 1.27 1.27)) (justify right bottom))
   )
@@
     (effects (font (size 1.27 1.27)) (justify left bottom))
   )
-  (label "MISO0" (at 110.49 74.93 180)
+  (label "SPI0_POCI0" (at 110.49 74.93 180)
     (effects (font (size 1.27 1.27)) (justify right bottom))
   )
@@
     (effects (font (size 1.27 1.27)) (justify right bottom))
   )
+  (label "SPI0_POCI0" (at 78.74 161.29 0)
+    (effects (font (size 1.27 1.27)) (justify left bottom))
+  )
   (label "PICO_PWM" (at 250.19 140.97 180)
     (effects (font (size 1.27 1.27)) (justify right bottom))
@@
     (effects (font (size 1.27 1.27)) (justify right bottom))
   )
-  (label "MISO0" (at 78.74 160.02 0)
-    (effects (font (size 1.27 1.27)) (justify left bottom))
-  )
   (label "PICO_DVI_CK+" (at 332.74 52.07 0)
     (effects (font (size 1.27 1.27)) (justify left bottom))
@@
     (effects (font (size 1.27 1.27)) (justify right bottom))
   )
-  (label "MOSI0" (at 36.83 160.02 0)
-    (effects (font (size 1.27 1.27)) (justify left bottom))
-  )
   (label "PICO_CEC" (at 250.19 105.41 180)
     (effects (font (size 1.27 1.27)) (justify right bottom))
@@
     (effects (font (size 1.27 1.27)) (justify left bottom))
   )
+  (label "SPI0_PICO0" (at 36.83 161.29 0)
+    (effects (font (size 1.27 1.27)) (justify left bottom))
+  )
   (label "PICO_UART0_RX" (at 250.19 82.55 180)
     (effects (font (size 1.27 1.27)) (justify right bottom))
@@
   (symbol (lib_id "Jumper:SolderJumper_3_Open") (at 92.71 156.21 0) (unit 1)
     (in_bom yes) (on_board yes) (fields_autoplaced)
-    (property "Reference" "JP3" (id 0) (at 92.71 149.86 0))
+    (property "Reference" "JP2" (id 0) (at 92.71 149.86 0))
     (property "Value" "SPI0_POCI" (id 1) (at 92.71 152.4 0))
     (property "Footprint" "Jumper:SolderJumper-3_P1.3mm_Open_RoundedPad1.0x1.5mm" (id 2) (at 92.71 156.21 0)
@@
   (symbol (lib_id "Jumper:SolderJumper_2_Open") (at 299.72 69.85 0) (unit 1)
     (in_bom yes) (on_board yes) (fields_autoplaced)
-    (property "Reference" "JP8" (id 0) (at 299.72 63.5 0))
+    (property "Reference" "JP4" (id 0) (at 299.72 63.5 0))
     (property "Value" "DVI_SCL" (id 1) (at 299.72 66.04 0))
     (property "Footprint" "Jumper:SolderJumper-2_P1.3mm_Open_RoundedPad1.0x1.5mm" (id 2) (at 299.72 69.85 0)
@@
       (effects (font (size 1.27 1.27)) hide)
     )
-    (property "Datasheet" "~" (id 3) (at 149.86 113.03 0)
+    (property "Datasheet" "https://datasheet.lcsc.com/lcsc/2103291203_Yangxing-Tech-X322512MSB4SI_C9002.pdf" (id 3) (at 149.86 113.03 0)
       (effects (font (size 1.27 1.27)) hide)
     )
@@
   (symbol (lib_id "Jumper:SolderJumper_2_Open") (at 299.72 59.69 0) (unit 1)
     (in_bom yes) (on_board yes) (fields_autoplaced)
-    (property "Reference" "JP7" (id 0) (at 299.72 53.34 0))
+    (property "Reference" "JP3" (id 0) (at 299.72 53.34 0))
     (property "Value" "DVI_CEC" (id 1) (at 299.72 55.88 0))
     (property "Footprint" "Jumper:SolderJumper-2_P1.3mm_Open_RoundedPad1.0x1.5mm" (id 2) (at 299.72 59.69 0)
@@
   (symbol (lib_id "Jumper:SolderJumper_2_Open") (at 299.72 80.01 0) (unit 1)
     (in_bom yes) (on_board yes) (fields_autoplaced)
-    (property "Reference" "JP9" (id 0) (at 299.72 73.66 0))
+    (property "Reference" "JP5" (id 0) (at 299.72 73.66 0))
     (property "Value" "DVI_SDA" (id 1) (at 299.72 76.2 0))
     (property "Footprint" "Jumper:SolderJumper-2_P1.3mm_Open_RoundedPad1.0x1.5mm" (id 2) (at 299.72 80.01 0)
@@
     )
     (path "/7a946772-8abf-40a2-b237-caac41608a67"
-      (reference "JP3") (unit 1) (value "SPI0_POCI") (footprint "Jumper:SolderJumper-3_P1.3mm_Open_RoundedPad1.0x1.5mm")
+      (reference "JP2") (unit 1) (value "SPI0_POCI") (footprint "Jumper:SolderJumper-3_P1.3mm_Open_RoundedPad1.0x1.5mm")
     )
     (path "/93702073-0a01-4e35-9305-8560c5685e9a"
-      (reference "JP7") (unit 1) (value "DVI_CEC") (footprint "Jumper:SolderJumper-2_P1.3mm_Open_RoundedPad1.0x1.5mm")
+      (reference "JP3") (unit 1) (value "DVI_CEC") (footprint "Jumper:SolderJumper-2_P1.3mm_Open_RoundedPad1.0x1.5mm")
     )
     (path "/816d84b4-262d-4b10-96cc-c865e194fe69"
-      (reference "JP8") (unit 1) (value "DVI_SCL") (footprint "Jumper:SolderJumper-2_P1.3mm_Open_RoundedPad1.0x1.5mm")
+      (reference "JP4") (unit 1) (value "DVI_SCL") (footprint "Jumper:SolderJumper-2_P1.3mm_Open_RoundedPad1.0x1.5mm")
     )
     (path "/99c0af06-3761-4a41-bdfe-96c9448a0497"
-      (reference "JP9") (unit 1) (value "DVI_SDA") (footprint "Jumper:SolderJumper-2_P1.3mm_Open_RoundedPad1.0x1.5mm")
+      (reference "JP5") (unit 1) (value "DVI_SDA") (footprint "Jumper:SolderJumper-2_P1.3mm_Open_RoundedPad1.0x1.5mm")
     )
     (path "/f6a99939-5049-4d29-bb1e-1b0361f8070e"
